Commit message: rbcar

File: bobcat/bobcat_description/urdf/bobcat.xacro (robot description, xacro)
@@ -113,4 +113,25 @@
       </collision>
     </link>
+        <link name="steering_wheel_fr_direction">
+        <inertial>
+      <mass value="5"/>
+      <origin rpy="0 0 0" xyz="0 0 0.1"/>
+      <inertia ixx="0.0395416666667" ixy="0" ixz="0" iyy="0.106208333333" iyz="0" izz="0.106208333333"/>
+    </inertial>
+      <visual>
+          <origin rpy="1.57079632679 0 0" xyz="0.5 0.36 0.08"/>
+          <!--geometry>
+            <mesh filename="package://bobcat_description/meshes/fr_wheel.stl" scale="0.001 0.001 0.001"/>
+          </geometry>
+          <material name="Black"/-->
+      </visual>
+            <collision>
+          <!--origin rpy="1.57079632679 0 0" xyz="0.5 0.36 0.08"/>
+          <geometry>
+            <mesh filename="package://bobcat_description/meshes/fr_wheel.stl" scale="0.001 0.001 0.001"/>
+          </geometry>
+          <material name="Black"/-->
+      </collision>
+    </link>
     <link name="steering_wheel_fl">
         <inertial>
@@ -134,4 +155,25 @@
       </collision>
     </link>
+        <link name="steering_wheel_fl_direction">
+        <inertial>
+      <mass value="5"/>
+      <origin rpy="0 0 0" xyz="0 0 0.1"/>
+      <inertia ixx="0.0395416666667" ixy="0" ixz="0" iyy="0.106208333333" iyz="0" izz="0.106208333333"/>
+    </inertial>
+      <visual>
+          <origin rpy="1.57079632679 0 0" xyz="-0.5 0.36 0.08"/>
+          <!--geometry>
+            <mesh filename="package://bobcat_description/meshes/fl_wheel.stl" scale="0.001 0.001 0.001"/>
+          </geometry>
+          <material name="Black"/-->
+      </visual>
+            <collision>
+          <!--origin rpy="1.57079632679 0 0" xyz="-0.5 0.36 0.08"/>
+          <geometry>
+            <mesh filename="package://bobcat_description/meshes/fl_wheel.stl" scale="0.001 0.001 0.001"/>
+          </geometry>
+          <material name="Black"/-->
+      </collision>
+    </link>
     <link name="steering_wheel_rr">
         <inertial>
@@ -176,29 +218,41 @@
       </collision>
     </link>
-       <joint name="base_link_joint" type="fixed">
+    <!--joint name="body_to_steering" type="fixed">
+        <parent link="chassis"/>
+        <child link="steering_subassem"/>
+        <origin xyz="0 0 0"/>
+    </joint>
+    <joint name="body_to_steering_col" type="fixed">
+        <parent link="chassis"/>
+        <child link="steering_col_subassem"/>
+        <origin xyz="0 0 0"/>
+    </joint-->
+           <joint name="base_link_joint" type="fixed">
       <parent link="base_link" />
       <child link="chassis" />
       <origin rpy="0 0 0" xyz="0 0 0" />
    </joint>
-    <!--joint name="body_to_steering" type="fixed">
-        <parent link="chassis"/>
-        <child link="steering_subassem"/>
-        <origin xyz="0 0 0"/>
-    </joint>
-    <joint name="body_to_steering_col" type="fixed">
-        <parent link="chassis"/>
-        <child link="steering_col_subassem"/>
-        <origin xyz="0 0 0"/>
-    </joint-->
+     <joint name="frw_to_steering_direction" type="revolute">
+        <parent link="chassis"/>
+        <child link="steering_wheel_fr_direction"/>
+        <origin xyz="-0.5 -0.35 -0.08" rpy="0 1.5708 0"/>
+        <limit effort="1000" velocity="1000" lower="-0.55" upper="0.55"/>
+    </joint>
         <joint name="frw_to_steering" type="continuous">
-        <parent link="chassis"/>
+        <parent link="steering_wheel_fr_direction"/>
         <child link="steering_wheel_fr"/>
-        <origin xyz="-0.5 -0.35 -0.08"/>
+        <origin xyz="0 0 0" rpy="0 -1.5708 0"/>
         <limit effort="1000" velocity="1000"/>
     </joint>
+  <joint name="flw_to_steering_direction" type="revolute">
+        <parent link="chassis"/>
+        <child link="steering_wheel_fl_direction"/>
+        <origin xyz="0.5 -0.35 -0.08" rpy="0 1.5708 0"/>
+        <limit effort="1000" velocity="1000" lower="-0.55" upper="0.55"/>
+    </joint>
         <joint name="flw_to_steering" type="continuous">
-        <parent link="chassis"/>
+        <parent link="steering_wheel_fl_direction"/>
         <child link="steering_wheel_fl"/>
-        <origin xyz="0.5 -0.35 -0.08"/>
+        <origin xyz="0 0 0" rpy="0 -1.5708 0"/>
         <limit effort="1000" velocity="1000"/>
     </joint>
