Commit message: agv works

File: agv/agv_description/urdf/agv.xacro (robot description, xacro)
@@ -34,120 +34,570 @@
     <material>Gazebo/Blue</material>
   </gazebo>
-  <link name="link_chassis">
-    <!-- pose and inertial -->
-    <pose>0 0 0.1 0 0 0</pose>
-    <inertial>
-      <mass value="5"/>
-      <origin rpy="0 0 0" xyz="0 0 0.1"/>
-      <inertia ixx="0.0395416666667" ixy="0" ixz="0" iyy="0.106208333333" iyz="0" izz="0.106208333333"/>
-    </inertial>
-    <collision name="collision_chassis">
-      <geometry>
-        <box size="0.5 0.3 0.07"/>
-      </geometry>
-    </collision>
-    <visual>
-      <origin rpy="0 0 0" xyz="0 0 0"/>
-      <geometry>
-        <box size="0.5 0.3 0.07"/>
+     <link name="base_link">
+      <visual>
+         <origin rpy="0 0 0" xyz="0 0 0" />
+      </visual>
+   </link>
+  <link name="chassis">
+    <!--pose>0 0 0.1 0 0 0</pose-->
+    <inertial>
+      <mass value="26"/>
+      <origin rpy="0 0 0" xyz="0 0 0"/>
+      <inertia ixx="0.000000001" ixy="0" ixz="0" iyy="0" iyz="0" izz="0"/>
+    </inertial>
+    <collision>
+      <geometry>
+        <box size="1.17 0.26 0.15"/>
+      </geometry>
+    </collision>
+    <visual>
+      <origin rpy="0 0 0" xyz="0 0 0"/>
+      <geometry>
+        <box size="1.17 0.26 0.15"/>
       </geometry>
       <material name="blue"/>
     </visual>
-    <!-- caster front -->
-    <collision name="caster_front_collision">
-      <origin rpy=" 0 0 0" xyz="0.35 0 -0.05"/>
-      <geometry>
-        <sphere radius="0.05"/>
-      </geometry>
-      <surface>
-        <friction>
-          <ode>
-            <mu>0</mu>
-            <mu2>0</mu2>
-            <slip1>1.0</slip1>
-            <slip2>1.0</slip2>
-          </ode>
-        </friction>
-      </surface>
-    </collision>
-    <visual name="caster_front_visual">
-      <origin rpy=" 0 0 0" xyz="0.2 0 -0.05"/>
-      <geometry>
-        <sphere radius="0.05"/>
-      </geometry>
-    </visual>
     </link>
   <!-- Create wheel right -->
-  <link name="link_right_wheel">
-    <inertial>
-      <mass value="0.2"/>
-      <origin rpy="0 1.5707 1.5707" xyz="0 0 0"/>
-      <inertia ixx="0.00052666666" ixy="0" ixz="0" iyy="0.00052666666" iyz="0" izz="0.001"/>
-    </inertial>
-    <collision name="link_right_wheel_collision">
-      <origin rpy="0 1.5707 1.5707" xyz="0 0 0" />
-      <geometry>
-        <cylinder length="0.04" radius="0.1"/>
-      </geometry>
-    </collision>
-    <visual name="link_right_wheel_visual">
-      <origin rpy="0 1.5707 1.5707" xyz="0 0 0"/>
-      <geometry>
-        <cylinder length="0.04" radius="0.1"/>
-      </geometry>
-    </visual>
+    <link name="wheel_1">
+    <inertial>
+      <mass value="0.5"/>
+      <origin rpy="0 0 0" xyz="0 0 0"/>
+      <inertia ixx="0.000000001" ixy="0" ixz="0" iyy="0" iyz="0" izz="0"/>
+    </inertial>
+    <collision>
+<origin rpy="0 1.57 0" xyz="0 0 0"/>
+      <geometry>
+        <cylinder length="0.1" radius="0.085"/>
+      </geometry>
+    </collision>
+    <visual>
+      <origin rpy="0 1.57 0" xyz="0 0 0"/>
+      <geometry>
+        <cylinder length="0.1" radius="0.085"/>
+      </geometry>
+      <material name="white"/>
+    </visual>
+    </link>
+        <link name="wheel_1_dir">
+     <inertial>
+      <mass value="0.5"/>
+      <origin rpy="0 0 0" xyz="0 0 0"/>
+      <inertia ixx="0.000000001" ixy="0" ixz="0" iyy="0" iyz="0" izz="0"/>
+    </inertial>
+    </link>
+        <link name="wheel_2">
+    <inertial>
+      <mass value="0.5"/>
+      <origin rpy="0 0 0" xyz="0 0 0"/>
+      <inertia ixx="0.000000001" ixy="0" ixz="0" iyy="0" iyz="0" izz="0"/>
+    </inertial>
+    <collision>
+<origin rpy="0 1.57 0" xyz="0 0 0"/>
+      <geometry>
+        <cylinder length="0.1" radius="0.085"/>
+      </geometry>
+    </collision>
+    <visual>
+      <origin rpy="0 1.57 0" xyz="0 0 0"/>
+      <geometry>
+        <cylinder length="0.1" radius="0.085"/>
+      </geometry>
+      <material name="white"/>
+    </visual>
+    </link>
+        <link name="wheel_2_dir">
+    <inertial>
+      <mass value="0.5"/>
+      <origin rpy="0 0 0" xyz="0 0 0"/>
+      <inertia ixx="0.000000001" ixy="0" ixz="0" iyy="0" iyz="0" izz="0"/>
+    </inertial>
+    </link>
+            <link name="wheel_3">
+    <inertial>
+      <mass value="0.5"/>
+      <origin rpy="0 0 0" xyz="0 0 0"/>
+      <inertia ixx="0.000000001" ixy="0" ixz="0" iyy="0" iyz="0" izz="0"/>
+    </inertial>
+    <collision>
+<origin rpy="0 1.57 0" xyz="0 0 0"/>
+      <geometry>
+        <cylinder length="0.1" radius="0.085"/>
+      </geometry>
+    </collision>
+    <visual>
+      <origin rpy="0 1.57 0" xyz="0 0 0"/>
+      <geometry>
+        <cylinder length="0.1" radius="0.085"/>
+      </geometry>
+      <material name="white"/>
+    </visual>
+    </link>
+        <link name="wheel_3_dir">
+    <inertial>
+      <mass value="0.5"/>
+      <origin rpy="0 0 0" xyz="0 0 0"/>
+      <inertia ixx="0.000000001" ixy="0" ixz="0" iyy="0" iyz="0" izz="0"/>
+    </inertial>
+    </link>
+                <link name="wheel_4">
+    <inertial>
+      <mass value="0.5"/>
+      <origin rpy="0 0 0" xyz="0 0 0"/>
+      <inertia ixx="0.000000001" ixy="0" ixz="0" iyy="0" iyz="0" izz="0"/>
+    </inertial>
+    <collision>
+<origin rpy="0 1.57 0" xyz="0 0 0"/>
+      <geometry>
+        <cylinder length="0.1" radius="0.085"/>
+      </geometry>
+    </collision>
+    <visual>
+      <origin rpy="0 1.57 0" xyz="0 0 0"/>
+      <geometry>
+        <cylinder length="0.1" radius="0.085"/>
+      </geometry>
+      <material name="white"/>
+    </visual>
+    </link>
+        <link name="wheel_4_dir">
+       <inertial>
+      <mass value="0.5"/>
+      <origin rpy="0 0 0" xyz="0 0 0"/>
+      <inertia ixx="0.000000001" ixy="0" ixz="0" iyy="0" iyz="0" izz="0"/>
+    </inertial>
+    </link>
+                <link name="wheel_5">
+    <inertial>
+      <mass value="0.5"/>
+      <origin rpy="0 0 0" xyz="0 0 0"/>
+      <inertia ixx="0.000000001" ixy="0" ixz="0" iyy="0" iyz="0" izz="0"/>
+    </inertial>
+    <collision>
+<origin rpy="0 1.57 0" xyz="0 0 0"/>
+      <geometry>
+        <cylinder length="0.1" radius="0.085"/>
+      </geometry>
+    </collision>
+    <visual>
+      <origin rpy="0 1.57 0" xyz="0 0 0"/>
+      <geometry>
+        <cylinder length="0.1" radius="0.085"/>
+      </geometry>
+      <material name="white"/>
+    </visual>
+    </link>
+        <link name="wheel_5_dir">
+   <inertial>
+      <mass value="0.5"/>
+      <origin rpy="0 0 0" xyz="0 0 0"/>
+      <inertia ixx="0.000000001" ixy="0" ixz="0" iyy="0" iyz="0" izz="0"/>
+    </inertial>
+    </link>
+                <link name="wheel_6">
+    <inertial>
+      <mass value="0.5"/>
+      <origin rpy="0 0 0" xyz="0 0 0"/>
+      <inertia ixx="0.000000001" ixy="0" ixz="0" iyy="0" iyz="0" izz="0"/>
+    </inertial>
+    <collision>
+<origin rpy="0 1.57 0" xyz="0 0 0"/>
+      <geometry>
+        <cylinder length="0.1" radius="0.085"/>
+      </geometry>
+    </collision>
+    <visual>
+      <origin rpy="0 1.57 0" xyz="0 0 0"/>
+      <geometry>
+        <cylinder length="0.1" radius="0.085"/>
+      </geometry>
+      <material name="white"/>
+    </visual>
+    </link>
+        <link name="wheel_6_dir">
+      <inertial>
+      <mass value="0.5"/>
+      <origin rpy="0 0 0" xyz="0 0 0"/>
+      <inertia ixx="0.000000001" ixy="0" ixz="0" iyy="0" iyz="0" izz="0"/>
+    </inertial>
+    </link>
+                <link name="wheel_7">
+    <inertial>
+      <mass value="0.5"/>
+      <origin rpy="0 0 0" xyz="0 0 0"/>
+      <inertia ixx="0.000000001" ixy="0" ixz="0" iyy="0" iyz="0" izz="0"/>
+    </inertial>
+    <collision>
+<origin rpy="0 1.57 0" xyz="0 0 0"/>
+      <geometry>
+        <cylinder length="0.1" radius="0.085"/>
+      </geometry>
+    </collision>
+    <visual>
+      <origin rpy="0 1.57 0" xyz="0 0 0"/>
+      <geometry>
+        <cylinder length="0.1" radius="0.085"/>
+      </geometry>
+      <material name="white"/>
+    </visual>
+    </link>
+        <link name="wheel_7_dir">
+     <inertial>
+      <mass value="0.5"/>
+      <origin rpy="0 0 0" xyz="0 0 0"/>
+      <inertia ixx="0.000000001" ixy="0" ixz="0" iyy="0" iyz="0" izz="0"/>
+    </inertial>
+    </link>
+                <link name="wheel_8">
+     <inertial>
+      <mass value="0.5"/>
+      <origin rpy="0 0 0" xyz="0 0 0"/>
+      <inertia ixx="0.000000001" ixy="0" ixz="0" iyy="0" iyz="0" izz="0"/>
+    </inertial>
+    <collision>
+    <origin rpy="0 1.57 0" xyz="0 0 0"/>
+      <geometry>
+        <cylinder length="0.1" radius="0.085"/>
+      </geometry>
+    </collision>
+    <visual>
+      <origin rpy="0 1.57 0" xyz="0 0 0"/>
+      <geometry>
+        <cylinder length="0.1" radius="0.085"/>
+      </geometry>
+      <material name="white"/>
+    </visual>
+    </link>
+        <link name="wheel_8_dir">
+    <inertial>
+      <mass value="0.5"/>
+      <origin rpy="0 0 0" xyz="0 0 0"/>
+      <inertia ixx="0.000000001" ixy="0" ixz="0" iyy="0" iyz="0" izz="0"/>
+    </inertial>
+    </link>
+  <!--   Joint for right wheel  -->
+  <joint name="joint_chassis" type="fixed">
+    <origin rpy="0 0 0" xyz="0 0 0"/>
+    <child link="chassis" />
+    <parent link="base_link"/>
+    <axis rpy="0 0 0" xyz="0 0 0"/>
+    <!--limit effort="10000" velocity="1000"/>
+    <joint_properties damping="1.0" friction="1.0" /-->
+  </joint>
+    <joint name="joint_wheel_1_dir" type="revolute">
+    <origin rpy="0 1.57 0" xyz="0.4 0.25 -0.05"/>
+    <child link="wheel_1_dir" />
+    <parent link="chassis"/>
+   <limit effort="1000" velocity="1000" lower="-0.55" upper="0.55"/>
+  </joint>
+    <joint name="joint_wheel_1" type="continuous">
+    <origin rpy="0 0 1.57" xyz="0 0 0"/>
+    <child link="wheel_1" />
+    <parent link="wheel_1_dir"/>
+   <limit effort="1000" velocity="1000"/>
+  </joint>
+      <joint name="joint_wheel_2_dir" type="revolute">
+    <origin rpy="0 1.57 0" xyz="0.13 0.25 -0.05"/>
+    <child link="wheel_2_dir" />
+    <parent link="chassis"/>
+   <limit effort="1000" velocity="1000" lower="-0.55" upper="0.55"/>
+  </joint>
+    <joint name="joint_wheel_2" type="continuous">
+    <origin rpy="0 0 1.57" xyz="0 0 0"/>
+    <child link="wheel_2" />
+    <parent link="wheel_2_dir"/>
+   <limit effort="1000" velocity="1000"/>
+  </joint>
+       <joint name="joint_wheel_3_dir" type="revolute">
+    <origin rpy="0 1.57 0" xyz="-0.13 0.25 -0.05"/>
+    <child link="wheel_3_dir" />
+    <parent link="chassis"/>
+   <limit effort="1000" velocity="1000" lower="-0.55" upper="0.55"/>
+  </joint>
+    <joint name="joint_wheel_3" type="continuous">
+    <origin rpy="0 0 1.57" xyz="0 0 0"/>
+    <child link="wheel_3" />
+    <parent link="wheel_3_dir"/>
+   <limit effort="1000" velocity="1000"/>
+  </joint>
+   <joint name="joint_wheel_4_dir" type="revolute">
+    <origin rpy="0 1.57 0" xyz="-0.4 0.25 -0.05"/>
+    <child link="wheel_4_dir" />
+    <parent link="chassis"/>
+   <limit effort="1000" velocity="1000" lower="-0.55" upper="0.55"/>
+  </joint>
+    <joint name="joint_wheel_4" type="continuous">
+    <origin rpy="0 0 1.57" xyz="0 0 0"/>
+    <child link="wheel_4" />
+    <parent link="wheel_4_dir"/>
+   <limit effort="1000" velocity="1000"/>
+  </joint>
+     <joint name="joint_wheel_5_dir" type="revolute">
+    <origin rpy="0 1.57 0" xyz="0.4 -0.25 -0.05"/>
+    <child link="wheel_5_dir" />
+    <parent link="chassis"/>
+   <limit effort="1000" velocity="1000" lower="-0.55" upper="0.55"/>
+  </joint>
+    <joint name="joint_wheel_5" type="continuous">
+    <origin rpy="0 0 1.57" xyz="0 0 0"/>
+    <child link="wheel_5" />
+    <parent link="wheel_5_dir"/>
+   <limit effort="1000" velocity="1000"/>
+  </joint>
+     <joint name="joint_wheel_6_dir" type="revolute">
+    <origin rpy="0 1.57 0" xyz="0.13 -0.25 -0.05"/>
+    <child link="wheel_6_dir" />
+    <parent link="chassis"/>
+   <limit effort="1000" velocity="1000" lower="-0.55" upper="0.55"/>
+  </joint>
+    <joint name="joint_wheel_6" type="continuous">
+    <origin rpy="0 0 1.57" xyz="0 0 0"/>
+    <child link="wheel_6" />
+    <parent link="wheel_6_dir"/>
+   <limit effort="1000" velocity="1000"/>
+  </joint>
+     <joint name="joint_wheel_7_dir" type="revolute">
+    <origin rpy="0 1.57 0" xyz="-0.13 -0.25 -0.05"/>
+    <child link="wheel_7_dir" />
+    <parent link="chassis"/>
+   <limit effort="1000" velocity="1000" lower="-0.55" upper="0.55"/>
+  </joint>
+    <joint name="joint_wheel_7" type="continuous">
+    <origin rpy="0 0 1.57" xyz="0 0 0"/>
+    <child link="wheel_7" />
+    <parent link="wheel_7_dir"/>
+   <limit effort="1000" velocity="1000"/>
+  </joint>
+     <joint name="joint_wheel_8_dir" type="revolute">
+    <origin rpy="0 1.57 0" xyz="-0.4 -0.25 -0.05"/>
+    <child link="wheel_8_dir" />
+    <parent link="chassis"/>
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
File: bobcat/bobcat_description/urdf/bobcat.xacro (robot description, xacro)
@@ -272,8 +272,8 @@
       <type>transmission_interface/SimpleTransmission</type>
       <joint name="frw_to_steering">
-        <hardwareInterface>EffortJointInterface</hardwareInterface>
+        <hardwareInterface>hardware_interface/EffortJointInterface</hardwareInterface>
       </joint>
       <actuator name="motor_frw_to_steering">
-        <hardwareInterface>EffortJointInterface</hardwareInterface>
+        <hardwareInterface>hardware_interface/EffortJointInterface</hardwareInterface>
         <mechanicalReduction>1</mechanicalReduction>
       </actuator>
@@ -282,8 +282,8 @@
       <type>transmission_interface/SimpleTransmission</type>
       <joint name="flw_to_steering">
-        <hardwareInterface>EffortJointInterface</hardwareInterface>
+        <hardwareInterface>hardware_interface/EffortJointInterface</hardwareInterface>
       </joint>
       <actuator name="motor_flw_to_steering">
-        <hardwareInterface>EffortJointInterface</hardwareInterface>
+        <hardwareInterface>hardware_interface/EffortJointInterface</hardwareInterface>
         <mechanicalReduction>1</mechanicalReduction>
       </actuator>
@@ -292,8 +292,8 @@
       <type>transmission_interface/SimpleTransmission</type>
       <joint name="body_to_rrw">
-        <hardwareInterface>EffortJointInterface</hardwareInterface>
+        <hardwareInterface>hardware_interface/EffortJointInterface</hardwareInterface>
       </joint>
       <actuator name="motor_body_to_rrw">
-        <hardwareInterface>EffortJointInterface</hardwareInterface>
+        <hardwareInterface>hardware_interface/EffortJointInterface</hardwareInterface>
         <mechanicalReduction>1</mechanicalReduction>
       </actuator>
@@ -302,14 +302,15 @@
       <type>transmission_interface/SimpleTransmission</type>
       <joint name="body_to_rlw">
-        <hardwareInterface>EffortJointInterface</hardwareInterface>
+        <hardwareInterface>hardware_interface/EffortJointInterface</hardwareInterface>
       </joint>
       <actuator name="motor_body_to_rlw">
-        <hardwareInterface>EffortJointInterface</hardwareInterface>
+        <hardwareInterface>hardware_interface/EffortJointInterface</hardwareInterface>
         <mechanicalReduction>1</mechanicalReduction>
       </actuator>
     </transmission>
   <gazebo>
-    <plugin name="gazebo_ros_control" filename="libgazebo_ros_control.so"/>
+    <plugin name="gazebo_ros_control" filename="libgazebo_ros_control.so">
     <robotNamespace>/bobcat</robotNamespace>
+    </plugin>
   </gazebo>
 </robot>
