Commit message: agv ackermann 8 wheeled

File: agv/agv_description/urdf/robot_2 (copy).xacro (robot description, xacro)
@@ -76,5 +76,5 @@
     </visual>
   </link>
-    <link name="link_right_wheel_dir">
+    <link name="right_steering">
     <inertial>
       <mass value="0.01"/>
@@ -320,7 +320,7 @@
     </sensor>
 </gazebo>
-  <joint name="joint_right_wheel_dir" type="revolute">
+  <joint name="right_steering_joint" type="revolute">
     <origin rpy="0 0 0" xyz="-0.4 0.25 -0.05"/>
-    <child link="link_right_wheel_dir" />
+    <child link="right_steering" />
     <parent link="link_chassis"/>
     <axis rpy="0 0 0" xyz="0 0 1"/>
@@ -332,5 +332,5 @@
     <origin rpy="0 0 0" xyz="0 0 0"/>
     <child link="link_right_wheel" />
-    <parent link="link_right_wheel_dir"/>
+    <parent link="right_steering"/>
     <limit effort="10000" velocity="1000"/>
     <axis rpy="0 0 0" xyz="0 1 0"/>
@@ -532,10 +532,10 @@
       </actuator>
     </transmission-->
-        <transmission name="tran_joint_right_wheel_dir">
-      <type>transmission_interface/SimpleTransmission</type>
-      <joint name="joint_right_wheel_dir">
-        <hardwareInterface>hardware_interface/EffortJointInterface</hardwareInterface>
-      </joint>
-      <actuator name="motor_joint_right_wheel_dir">
+        <transmission name="tran_right_steering_joint">
+      <type>transmission_interface/SimpleTransmission</type>
+      <joint name="right_steering_joint">
+        <hardwareInterface>hardware_interface/EffortJointInterface</hardwareInterface>
+      </joint>
+      <actuator name="motor_right_steering_joint">
         <hardwareInterface>hardware_interface/EffortJointInterface</hardwareInterface>
         <mechanicalReduction>1</mechanicalReduction>

File: agv/agv_description/urdf/robot_2_no_dir.xacro (robot description, xacro)
@@ -278,18 +278,19 @@
   </joint>
   <!--   Joint for right wheel  -->
-<!--gazebo>
-    <plugin filename="libgazebo_ros_diff_drive.so" name="differential_drive_controller">
-      <alwaysOn>true</alwaysOn>
-      <updateRate>20</updateRate>
-      <leftJoint>joint_left_wheel</leftJoint>
-      <rightJoint>joint_right_wheel</rightJoint>
-      <wheelSeparation>0.4</wheelSeparation>
-      <wheelDiameter>0.2</wheelDiameter>
-      <torque>0.1</torque>
-      <commandTopic>cmd_vel</commandTopic>
-      <odometryTopic>odom</odometryTopic>
-      <odometryFrame>odom</odometryFrame>
-      <robotBaseFrame>link_chassis</robotBaseFrame>
-    </plugin>
-  </gazebo-->
+      <!--gazebo>
+        <plugin name="agv_multi_controller" filename="libdiffdrive_plugin_multi_wheel.so">
+        <commandTopic>cmd_vel</commandTopic>
+        <rightJoints>joint_right_wheel joint_right_wheel_2 joint_right_wheel_3 joint_right_wheel_4</rightJoints>
+        <leftJoints>joint_left_wheel joint_left_wheel_2 joint_left_wheel_3 joint_left_wheel_4</leftJoints>
+        <odometryTopic>world</odometryTopic>
+        <odometryFrame>world</odometryFrame>
+        <odometryRate>20.0</odometryRate>
+	<publishOdometryTf>true</publishOdometryTf>
+        <publishOdometryMsg>false</publishOdometryMsg>
+        <robotBaseFrame>link_chassis</robotBaseFrame>
+        </plugin>
+    </gazebo-->
+  <gazebo>
+    <plugin name="gazebo_ros_control" filename="libgazebo_ros_control.so"/>
+  </gazebo>
 </robot>
